Commit message: new models

File: robotiq_hande_gripper_description/urdf/robotiq_hande.urdf.xacro (robot description, xacro)
@@ -2,5 +2,31 @@
 <robot xmlns:xacro="http://ros.org/wiki/xacro">
   <xacro:macro name="robotiq_hande"  params="prefix MAC">
-    <link name="${prefix}robotiq_hande_base_link">
+    <link name="${prefix}coupling_link">
+      <inertial>
+        <origin xyz="0 0 0.00835" rpy="0 0 0" />
+        <mass value="0.1305" />
+        <inertia ixx="1017560E-9" ixy="0" ixz="2235E-9" iyy="1028041E-9" iyz="0" izz="489810E-9" />
+      </inertial>
+      <visual>
+        <origin xyz="0 0 0" rpy="0 0 0" />
+        <geometry>
+          <mesh filename="package://robotiq_hande_gripper_description/meshes/coupling.dae" scale="0.001 0.001 0.001"/>
+        </geometry>
+        <material name="Gazebo/Black">
+          <color rgba="1 1 1 1" />
+        </material>
+      </visual>
+      <collision>
+        <origin xyz="0 0 0" rpy="0 0 0" />
+        <geometry>
+          <mesh filename="package://robotiq_hande_gripper_description/meshes/coupling.dae" scale="0.001 0.001 0.001"/>
+        </geometry>
+      </collision>
+    </link>
+    <gazebo reference="${prefix}coupling_link">
+      <material>Gazebo/Black</material>
+      <selfCollide>True</selfCollide>
+    </gazebo>
+    <link name="${prefix}base_link">
       <inertial>
         <origin xyz="0 0 0.04607" rpy="0 0 0" />
@@ -24,5 +50,5 @@
       </collision>
     </link>
-    <gazebo reference="${prefix}robotiq_hande_base_link">
+    <gazebo reference="${prefix}base_link">
       <material>Gazebo/Black</material>
       <selfCollide>True</selfCollide>
@@ -80,7 +106,12 @@
       <selfCollide>True</selfCollide>
     </gazebo>
+    <joint name="${prefix}coupling_base" type="fixed">
+      <origin rpy="0 0 0" xyz="0 0 0.092"/>
+      <parent link="${prefix}coupling_link"/>
+      <child link="${prefix}base_link"/>
+    </joint>
     <joint name="${prefix}joint_finger" type="prismatic">
-      <origin rpy="0 0 0" xyz="0 0 0.099"/>
-      <parent link="${prefix}robotiq_hande_base_link"/>
+      <origin rpy="0 0 0" xyz="0 0 0.014"/>
+      <parent link="${prefix}base_link"/>
       <child link="${prefix}left_finger"/>
       <axis xyz="-1 0 0"/>
@@ -88,6 +119,6 @@
     </joint>
     <joint name="robotiq_hande_base_to_${prefix}right_finger" type="prismatic">
-      <origin rpy="0 0 0" xyz="0 0 0.099"/>
-      <parent link="${prefix}robotiq_hande_base_link"/>
+      <origin rpy="0 0 0" xyz="0 0 0.014"/>
+      <parent link="${prefix}base_link"/>
       <child link="${prefix}right_finger"/>
       <axis xyz="1 0 0"/>

File: ur_description/urdf/ur-hande.xacro (robot description, xacro)
@@ -28,12 +28,11 @@
      safety_pos_margin="$(arg safety_pos_margin)"
      safety_k_position="$(arg safety_k_position)"/>
-   <!-- TODO: Add flange -->
    <!-- gripper -->
    <xacro:include filename="$(find robotiq_hande_gripper_description)/urdf/robotiq_hande.urdf.xacro"/>
    <xacro:robotiq_hande prefix="hande_" MAC="_000000000004"/>
    <joint name="tool0_robotiq_adapter" type="fixed">
-    <origin rpy="0 0 0" xyz="0 0 0.0167"/>
+    <origin rpy="0 0 0" xyz="0 0 0.0035"/>
     <parent link="tool0"/>
-    <child link="hande_robotiq_hande_base_link"/>
+    <child link="hande_coupling_link"/>
   </joint>
 </robot>

Commit message: adjust params for moveit and rmp

File: robotiq_hande_gripper_description/urdf/robotiq_hande.urdf.xacro (robot description, xacro)
@@ -111,5 +111,5 @@
       <child link="${prefix}base_link"/>
     </joint>
-    <joint name="${prefix}joint_finger" type="prismatic">
+    <joint name="${prefix}left_finger_joint" type="fixed">
       <origin rpy="0 0 0" xyz="0 0 0.014"/>
       <parent link="${prefix}base_link"/>
@@ -118,5 +118,5 @@
       <limit effort="130" lower="0" upper="0.025" velocity="0.15"/>
     </joint>
-    <joint name="robotiq_hande_base_to_${prefix}right_finger" type="prismatic">
+    <joint name="${prefix}right_finger_joint" type="fixed">
       <origin rpy="0 0 0" xyz="0 0 0.014"/>
       <parent link="${prefix}base_link"/>
@@ -124,5 +124,5 @@
       <axis xyz="1 0 0"/>
       <limit effort="130" lower="0" upper="0.025" velocity="0.15"/>
-      <mimic joint="${prefix}joint_finger" multiplier="1" offset="0"/>
+      <mimic joint="${prefix}left_finger_joint" multiplier="1" offset="0"/>
     </joint>
   </xacro:macro>

File: ur_description/urdf/ur-hande.xacro (robot description, xacro)
@@ -1,11 +1,11 @@
 <?xml version="1.0"?>
-<robot xmlns:xacro="http://wiki.ros.org/xacro" name="$(arg robot_model)_robot">
+<robot xmlns:xacro="http://wiki.ros.org/xacro" name="ur5e_robot">
    <!-- import main macro -->
    <xacro:include filename="$(find ur_description)/urdf/inc/ur_macro.xacro"/>
    <!-- parameters -->
-   <xacro:arg name="joint_limit_params" default=""/>
-   <xacro:arg name="kinematics_params" default=""/>
-   <xacro:arg name="physical_params" default=""/>
-   <xacro:arg name="visual_params" default=""/>
+   <xacro:arg name="joint_limit_params" default="$(find ur_description)/config/ur5e/joint_limits.yaml"/>
+   <xacro:arg name="kinematics_params" default="$(find ur_description)/config/ur5e/default_kinematics.yaml"/>
+   <xacro:arg name="physical_params" default="$(find ur_description)/config/ur5e/physical_parameters.yaml"/>
+   <xacro:arg name="visual_params" default="$(find ur_description)/config/ur5e/visual_parameters.yaml"/>
    <!-- legal values:
          - hardware_interface/PositionJointInterface
@@ -32,14 +32,14 @@
    <xacro:robotiq_hande prefix="hande_" MAC="_000000000004"/>
    <joint name="tool0_robotiq_adapter" type="fixed">
-    <origin rpy="0 0 0" xyz="0 0 0.0035"/>
-    <parent link="tool0"/>
-    <child link="hande_coupling_link"/>
-  </joint>
-  <!-- tool_center_point -->
-  <link name="tcp_link"/>
-  <joint name="tcp_joint" type="fixed">
-    <origin rpy="0 0 0" xyz="0 0 0.157"/>
-    <parent link="tool0"/>
+     <origin rpy="0 0 0" xyz="0 0 0.0035"/>
+     <parent link="tool0"/>
+     <child link="hande_coupling_link"/>
+   </joint>
+   <!-- tool_center_point -->
+   <link name="tcp_link"/>
+   <joint name="tcp_joint" type="fixed">
+    <origin rpy="0 0 0" xyz="0 0 0.0615"/>
+    <parent link="hande_base_link"/>
     <child link="tcp_link"/>
-  </joint>
+   </joint>
 </robot>
