Commit message: name changes in hande_world and hande.urdf

File: robotiq_hande_gripper_description/urdf/robotiq_hande.urdf (robot description, URDF)
Before this commit: robot robotiq_hande, 4 links, 3 joints
Links:
- removed link hande_robotiq_hande_base_link
- added link hande_base_link, mass 0.86387; collision mesh filename=package://robotiq_hande_gripper_description/meshes/hand-e.d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 scale=0.001 0.001 0.001; visual mesh filename=package://robotiq_hande_gripper_description/meshes/hand-e.d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 scale=0.001 0.001 0.001

File: robotiq_hande_gripper_description/urdf/robotiq_hande_world.urdf.xacro (robot description, xacro)
@@ -8,5 +8,5 @@
     <origin rpy="0 0 0" xyz="0 0 0.5"/>
     <parent link="world"/>
-    <child link="hande_robotiq_hande_base_link"/>
+    <child link="hande_base_link"/>
   </joint>
   <gazebo>
