Commit message: added ur3 virtual joints

File: robotiq_hande_gripper_description/urdf/ur-hande.xacro (robot description, xacro)
@@ -47,5 +47,5 @@
       <link name="virtual_shoulder_link"/>
       <joint name="virtual_shoulder_joint" type="fixed">
-          <origin rpy="0 0 0" xyz="0 -0.135 0"/>
+          <origin rpy="0 0 0" xyz="0 -0.138 0"/>
           <parent link="shoulder_link"/>
           <child link="virtual_shoulder_link"/>
@@ -53,5 +53,5 @@
       <link name="virtual_forearm_link"/>
       <joint name="virtual_forearm_joint" type="fixed">
-          <origin rpy="0 0 0" xyz="0 0 0.135"/>
+          <origin rpy="0 0 0" xyz="0 0 0.138"/>
           <parent link="forearm_link"/>
           <child link="virtual_forearm_link"/>
@@ -59,5 +59,26 @@
       <link name="virtual_wrist_1_link"/>
       <joint name="virtual_wrist_1_joint" type="fixed">
-          <origin rpy="0 0 0" xyz="0 0 -0.13"/>
+          <origin rpy="0 0 0" xyz="0 0 -0.127"/>
+          <parent link="wrist_1_link"/>
+          <child link="virtual_wrist_1_link"/>
+      </joint>
+    </xacro:if>
+    <xacro:if value="${'$(arg robot_model)' == 'ur3e_robot'}">
+      <!-- virtual joints for RMPs-->
+      <link name="virtual_shoulder_link"/>
+      <joint name="virtual_shoulder_joint" type="fixed">
+          <origin rpy="0 0 0" xyz="0 -0.12 0"/>
+          <parent link="shoulder_link"/>
+          <child link="virtual_shoulder_link"/>
+      </joint>
+      <link name="virtual_forearm_link"/>
+      <joint name="virtual_forearm_joint" type="fixed">
+          <origin rpy="0 0 0" xyz="0 0 0.12"/>
+          <parent link="forearm_link"/>
+          <child link="virtual_forearm_link"/>
+      </joint>
+      <link name="virtual_wrist_1_link"/>
+      <joint name="virtual_wrist_1_joint" type="fixed">
+          <origin rpy="0 0 0" xyz="0 0 -0.12"/>
           <parent link="wrist_1_link"/>
           <child link="virtual_wrist_1_link"/>
