Commit message: Add tcp_link to xacro

File: ur_description/urdf/ur-hande.xacro (robot description, xacro)
@@ -36,3 +36,10 @@
     <child link="hande_coupling_link"/>
   </joint>
+  <!-- tool_center_point -->
+  <link name="tcp_link"/>
+  <joint name="tcp_joint" type="fixed">
+    <origin rpy="0 0 0" xyz="0 0 0.157"/>
+    <parent link="tool0"/>
+    <child link="tcp_link"/>
+  </joint>
 </robot>

Commit message: small changes on sensor_moveit.yaml

File: ur_description/urdf/ur-hande.xacro (robot description, xacro)
@@ -39,7 +39,7 @@
    <link name="tcp_link"/>
    <joint name="tcp_joint" type="fixed">
-    <origin rpy="0 0 0" xyz="0 0 0.0615"/>
-    <parent link="hande_base_link"/>
-    <child link="tcp_link"/>
+     <origin rpy="0 0 0" xyz="0 0 0.0615"/>
+     <parent link="hande_base_link"/>
+     <child link="tcp_link"/>
    </joint>
 </robot>
